File: power/powerboard.sch (EAGLE design)
At the start: 29 parts, among them Q1 IRFB7430, Q2 IRFB7430, Q3 IRFB7430, T1 BCP56, T2 BCP53, T3 BCP56, T4 BCP53, T5 BCP56, T6 BCP53

Commit message: power brd
Parts:
- added F2: (no value), fuse:SH22,5
- added OUT1, OUT2, OUT3, PWRIN1, PWRIN2: (no value), Terminal_Blocks_Connectors_rev15e:691244610002
Connections:
- removed net 12VIN: F1.1
- new net 12V2: F2.2, OK3.COL, OUT3.1, R11.2
- new net 12VIN1: F1.1, PWRIN1.1
- new net 12VIN2: F2.1, PWRIN2.1
- net 12V: now also OUT1.1, OUT2.1; no longer OK3.COL, R11.2
- net PCH1-2: now also OUT1.2
- net PCH2-2: now also OUT2.2
- net PCH3-2: now also OUT3.2
- net PWRGND: now also PWRIN1.2, PWRIN2.2
Changed lines of the file:
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@@
 <part name="R15" library="rcl" deviceset="R-EU_" device="R0805" value="10K"/>
 <part name="F1" library="fuse" deviceset="SH22,5" device=""/>
+<part name="F2" library="fuse" deviceset="SH22,5" device=""/>
+<part name="PWRIN1" library="Terminal_Blocks_Connectors_rev15e" deviceset="691244610002" device=""/>
+<part name="PWRIN2" library="Terminal_Blocks_Connectors_rev15e" deviceset="691244610002" device=""/>
+<part name="OUT1" library="Terminal_Blocks_Connectors_rev15e" deviceset="691244610002" device=""/>
+<part name="OUT2" library="Terminal_Blocks_Connectors_rev15e" deviceset="691244610002" device=""/>
+<part name="OUT3" library="Terminal_Blocks_Connectors_rev15e" deviceset="691244610002" device=""/>
 </parts>
 <sheets>
@@
 <instance part="R15" gate="G$1" x="40.64" y="-48.26" rot="R90"/>
 <instance part="F1" gate="1" x="73.66" y="124.46"/>
+<instance part="F2" gate="1" x="73.66" y="119.38"/>
+<instance part="PWRIN1" gate="G$1" x="132.08" y="106.68"/>
+<instance part="PWRIN2" gate="G$1" x="132.08" y="99.06"/>
+<instance part="OUT1" gate="G$1" x="132.08" y="83.82"/>
+<instance part="OUT2" gate="G$1" x="132.08" y="76.2"/>
+<instance part="OUT3" gate="G$1" x="132.08" y="68.58"/>
 </instances>
 <busses>
@@
 <wire x1="40.64" y1="-58.42" x2="71.12" y2="-58.42" width="0.1524" layer="91"/>
 </segment>
+<segment>
+<pinref part="PWRIN2" gate="G$1" pin="2"/>
+<wire x1="127" y1="96.52" x2="124.46" y2="96.52" width="0.1524" layer="91"/>
+<pinref part="PWRIN1" gate="G$1" pin="2"/>
+<wire x1="124.46" y1="96.52" x2="119.38" y2="96.52" width="0.1524" layer="91"/>
+<wire x1="127" y1="104.14" x2="124.46" y2="104.14" width="0.1524" layer="91"/>
+<wire x1="124.46" y1="104.14" x2="124.46" y2="96.52" width="0.1524" layer="91"/>
+<wire x1="119.38" y1="96.52" x2="119.38" y2="93.98" width="0.1524" layer="91"/>
+<junction x="124.46" y="96.52"/>
+<label x="119.38" y="91.44" size="1.778" layer="95"/>
+</segment>
 </net>
 <net name="N$3" class="0">
@@
 <wire x1="25.4" y1="73.66" x2="22.86" y2="73.66" width="0.1524" layer="91"/>
 <wire x1="25.4" y1="88.9" x2="25.4" y2="73.66" width="0.1524" layer="91"/>
-<pinref part="OK3" gate="G$1" pin="COL"/>
-<wire x1="25.4" y1="58.42" x2="22.86" y2="58.42" width="0.1524" layer="91"/>
-<wire x1="25.4" y1="73.66" x2="25.4" y2="58.42" width="0.1524" layer="91"/>
 <junction x="25.4" y="88.9"/>
-<junction x="25.4" y="73.66"/>
 </segment>
 <segment>
@@
 </segment>
 <segment>
-<pinref part="R11" gate="G$1" pin="2"/>
-<wire x1="71.12" y1="-15.24" x2="71.12" y2="-17.78" width="0.1524" layer="91"/>
-<label x="66.04" y="-15.24" size="1.778" layer="95"/>
-</segment>
-<segment>
 <pinref part="F1" gate="1" pin="2"/>
 <wire x1="78.74" y1="124.46" x2="88.9" y2="124.46" width="0.1524" layer="91"/>
 <label x="91.44" y="124.46" size="1.778" layer="95"/>
 </segment>
+<segment>
+<pinref part="OUT1" gate="G$1" pin="1"/>
+<wire x1="127" y1="83.82" x2="124.46" y2="83.82" width="0.1524" layer="91"/>
+<wire x1="124.46" y1="83.82" x2="119.38" y2="83.82" width="0.1524" layer="91"/>
+<wire x1="124.46" y1="83.82" x2="124.46" y2="76.2" width="0.1524" layer="91"/>
+<pinref part="OUT2" gate="G$1" pin="1"/>
+<wire x1="124.46" y1="76.2" x2="127" y2="76.2" width="0.1524" layer="91"/>
+<junction x="124.46" y="83.82"/>
+<label x="114.3" y="83.82" size="1.778" layer="95"/>
+</segment>
 </net>
 <net name="N$8" class="0">
@@
 <wire x1="93.98" y1="86.36" x2="93.98" y2="91.44" width="0.1524" layer="91"/>
 <label x="96.52" y="91.44" size="1.778" layer="95"/>
+</segment>
+<segment>
+<pinref part="OUT1" gate="G$1" pin="2"/>
+<wire x1="127" y1="81.28" x2="119.38" y2="81.28" width="0.1524" layer="91"/>
+<label x="111.76" y="81.28" size="1.778" layer="95"/>
 </segment>
 </net>
@@
 <label x="96.52" y="27.94" size="1.778" layer="95"/>
 </segment>
+<segment>
+<pinref part="OUT2" gate="G$1" pin="2"/>
+<wire x1="127" y1="73.66" x2="119.38" y2="73.66" width="0.1524" layer="91"/>
+<label x="111.76" y="73.66" size="1.778" layer="95"/>
+</segment>
 </net>
 <net name="PCH3-2" class="0">
@@
 <wire x1="93.98" y1="-38.1" x2="93.98" y2="-33.02" width="0.1524" layer="91"/>
 <label x="96.52" y="-33.02" size="1.778" layer="95"/>
+</segment>
+<segment>
+<pinref part="OUT3" gate="G$1" pin="2"/>
+<wire x1="127" y1="66.04" x2="119.38" y2="66.04" width="0.1524" layer="91"/>
+<label x="111.76" y="66.04" size="1.778" layer="95"/>
 </segment>
 </net>
@@
 </segment>
 </net>
-<net name="12VIN" class="0">
+<net name="12VIN1" class="0">
 <segment>
 <pinref part="F1" gate="1" pin="1"/>
@@
 <label x="53.34" y="124.46" size="1.778" layer="95"/>
 </segment>
-</net>
+<segment>
+<pinref part="PWRIN1" gate="G$1" pin="1"/>
+<wire x1="127" y1="106.68" x2="119.38" y2="106.68" width="0.1524" layer="91"/>
+<label x="109.22" y="106.68" size="1.778" layer="95"/>
+</segment>
+</net>
+<net name="12VIN2" class="0">
+<segment>
+<pinref part="F2" gate="1" pin="1"/>
+<wire x1="68.58" y1="119.38" x2="60.96" y2="119.38" width="0.1524" layer="91"/>
+<label x="53.34" y="119.38" size="1.778" layer="95"/>
+</segment>
+<segment>
+<pinref part="PWRIN2" gate="G$1" pin="1"/>
+<wire x1="127" y1="99.06" x2="119.38" y2="99.06" width="0.1524" layer="91"/>
+<label x="109.22" y="99.06" size="1.778" layer="95"/>
+</segment>
+</net>
+<net name="12V2" class="0">
+<segment>
+<pinref part="F2" gate="1" pin="2"/>
+<wire x1="78.74" y1="119.38" x2="88.9" y2="119.38" width="0.1524" layer="91"/>
+<label x="91.44" y="119.38" size="1.778" layer="95"/>
+</segment>
+<segment>
+<pinref part="R11" gate="G$1" pin="2"/>
+<wire x1="71.12" y1="-15.24" x2="71.12" y2="-17.78" width="0.1524" layer="91"/>
+<label x="66.04" y="-15.24" size="1.778" layer="95"/>
+</segment>
+<segment>
+<pinref part="OUT3" gate="G$1" pin="1"/>
+<wire x1="127" y1="68.58" x2="119.38" y2="68.58" width="0.1524" layer="91"/>
+<label x="111.76" y="68.58" size="1.778" layer="95"/>
+</segment>
+<segment>
+<pinref part="OK3" gate="G$1" pin="COL"/>
+<wire x1="25.4" y1="58.42" x2="22.86" y2="58.42" width="0.1524" layer="91"/>
+<label x="25.4" y="58.42" size="1.778" layer="95"/>
+</segment>
+</net>
